Commit message: Added launch script and fixed bugs in order to be able to launch both RVIZ and Gazebo simulation at the same time.

File: src/gecko_robot/model/onshape_robot.xacro (robot description, xacro)
@@ -27,5 +27,5 @@
       <origin xyz="0.127962 0.0712341 -0.00962078" rpy="0 -0 0"/>
       <geometry>
-        <mesh filename="package://gecko_robot/model/base_link.stl"/>
+        <mesh filename="package://gecko_robot/meshes/base_link.stl"/>
       </geometry>
       <material name="base_link_material">
@@ -36,5 +36,5 @@
       <origin xyz="0.127962 0.0712341 -0.00962078" rpy="0 -0 0"/>
       <geometry>
-        <mesh filename="package://gecko_robot/model/base_link.stl"/>
+        <mesh filename="package://gecko_robot/meshes/base_link.stl"/>
       </geometry>
     </collision>
@@ -51,5 +51,5 @@
       <origin xyz="0 -2.77556e-17 0.0075" rpy="3.14159 -6.16298e-33 -2.42375e-18"/>
       <geometry>
-        <mesh filename="package://gecko_robot/model/leg.stl"/>
+        <mesh filename="package://gecko_robot/meshes/leg.stl"/>
       </geometry>
       <material name="leg_material">
@@ -60,5 +60,5 @@
       <origin xyz="0 -2.77556e-17 0.0075" rpy="3.14159 -6.16298e-33 -2.42375e-18"/>
       <geometry>
-        <mesh filename="package://gecko_robot/model/leg.stl"/>
+        <mesh filename="package://gecko_robot/meshes/leg.stl"/>
       </geometry>
     </collision>
@@ -83,5 +83,5 @@
       <origin xyz="-5.55112e-17 -5.55112e-17 0.0075" rpy="-3.14159 1.32734e-33 -2.95341e-17"/>
       <geometry>
-        <mesh filename="package://gecko_robot/model/leg.stl"/>
+        <mesh filename="package://gecko_robot/meshes/leg.stl"/>
       </geometry>
       <material name="leg_2_material">
@@ -92,5 +92,5 @@
       <origin xyz="-5.55112e-17 -5.55112e-17 0.0075" rpy="-3.14159 1.32734e-33 -2.95341e-17"/>
       <geometry>
-        <mesh filename="package://gecko_robot/model/leg.stl"/>
+        <mesh filename="package://gecko_robot/meshes/leg.stl"/>
       </geometry>
     </collision>
@@ -115,5 +115,5 @@
       <origin xyz="0 0 0.0075" rpy="3.14159 -7.70372e-34 -4.01774e-17"/>
       <geometry>
-        <mesh filename="package://gecko_robot/model/leg.stl"/>
+        <mesh filename="package://gecko_robot/meshes/leg.stl"/>
       </geometry>
       <material name="leg_3_material">
@@ -124,5 +124,5 @@
       <origin xyz="0 0 0.0075" rpy="3.14159 -7.70372e-34 -4.01774e-17"/>
       <geometry>
-        <mesh filename="package://gecko_robot/model/leg.stl"/>
+        <mesh filename="package://gecko_robot/meshes/leg.stl"/>
       </geometry>
     </collision>
@@ -147,5 +147,5 @@
       <origin xyz="-1.38778e-17 -1.38778e-17 0.0075" rpy="3.14159 2.18953e-47 1.9666e-18"/>
       <geometry>
-        <mesh filename="package://gecko_robot/model/leg.stl"/>
+        <mesh filename="package://gecko_robot/meshes/leg.stl"/>
       </geometry>
       <material name="leg_4_material">
@@ -156,5 +156,5 @@
       <origin xyz="-1.38778e-17 -1.38778e-17 0.0075" rpy="3.14159 2.18953e-47 1.9666e-18"/>
       <geometry>
-        <mesh filename="package://gecko_robot/model/leg.stl"/>
+        <mesh filename="package://gecko_robot/meshes/leg.stl"/>
       </geometry>
     </collision>
